File: memory/memory.kicad_sch (KiCad schematic)
At the start: 6 parts, among them J1 Conn_01x02, J2 Conn_01x15, J3 Conn_01x08, J4 Conn_01x06, U1 28C256

Commit message: Memory board
Parts:
- U1: footprint Package_DIP:DIP-28_W15.24mm_LongPads -> Socket:DIP_Socket-28_W11.9_W12.7_W15.24_W17.78_W18.5_3M_228-1277-00-0602J
Connections:
- net GND: now also J4.2 (Pin_2); no longer J4.4 (Pin_4)
- net a14: now also J4.4 (Pin_4); no longer J4.2 (Pin_2)
Changed lines of the file:
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@@
     (stroke (width 0) (type default) (color 0 0 0 0))
   )
-  (wire (pts (xy 106.68 78.74) (xy 106.68 91.44))
+  (wire (pts (xy 106.68 78.74) (xy 106.68 86.36))
     (stroke (width 0) (type default) (color 0 0 0 0))
   )
@@
     (stroke (width 0) (type default) (color 0 0 0 0))
   )
-  (wire (pts (xy 97.79 86.36) (xy 111.76 86.36))
-    (stroke (width 0) (type default) (color 0 0 0 0))
-  )
   (wire (pts (xy 151.13 43.18) (xy 153.67 43.18))
     (stroke (width 0) (type default) (color 0 0 0 0))
@@
     (stroke (width 0) (type default) (color 0 0 0 0))
   )
-  (wire (pts (xy 97.79 91.44) (xy 106.68 91.44))
+  (wire (pts (xy 97.79 86.36) (xy 106.68 86.36))
     (stroke (width 0) (type default) (color 0 0 0 0))
   )
@@
     (stroke (width 0) (type default) (color 0 0 0 0))
   )
+  (wire (pts (xy 97.79 91.44) (xy 111.76 91.44))
+    (stroke (width 0) (type default) (color 0 0 0 0))
+  )
   (wire (pts (xy 35.56 95.25) (xy 38.1 95.25))
     (stroke (width 0) (type default) (color 0 0 0 0))
@@
     (effects (font (size 1.27 1.27)) (justify left bottom))
   )
-  (label "a14" (at 101.6 91.44 0)
+  (label "a14" (at 101.6 86.36 0)
     (effects (font (size 1.27 1.27)) (justify left bottom))
   )
@@
     (pin "2")
   )
-  (symbol (lib_id "power:GND") (at 111.76 86.36 0) (unit 1)
-    (in_bom yes) (on_board yes) (fields_autoplaced)
-    (property "Reference" "#PWR0104" (id 0) (at 111.76 92.71 0)
-      (effects (font (size 1.27 1.27)) hide)
-    )
-    (property "Value" "GND" (id 1) (at 111.76 91.44 0))
-    (property "Footprint" "" (id 2) (at 111.76 86.36 0)
-      (effects (font (size 1.27 1.27)) hide)
-    )
-    (property "Datasheet" "" (id 3) (at 111.76 86.36 0)
+  (symbol (lib_id "power:GND") (at 111.76 91.44 0) (unit 1)
+    (in_bom yes) (on_board yes) (fields_autoplaced)
+    (property "Reference" "#PWR0104" (id 0) (at 111.76 97.79 0)
+      (effects (font (size 1.27 1.27)) hide)
+    )
+    (property "Value" "GND" (id 1) (at 111.76 96.52 0))
+    (property "Footprint" "" (id 2) (at 111.76 91.44 0)
+      (effects (font (size 1.27 1.27)) hide)
+    )
+    (property "Datasheet" "" (id 3) (at 111.76 91.44 0)
       (effects (font (size 1.27 1.27)) hide)
     )
@@
   (symbol (lib_id "power:+5V") (at 187.96 57.15 0) (unit 1)
     (in_bom yes) (on_board yes) (fields_autoplaced)
-    (property "Reference" "#PWR?" (id 0) (at 187.96 60.96 0)
+    (property "Reference" "#PWR0107" (id 0) (at 187.96 60.96 0)
       (effects (font (size 1.27 1.27)) hide)
     )
@@
   (symbol (lib_id "power:GND") (at 187.96 71.12 0) (unit 1)
     (in_bom yes) (on_board yes) (fields_autoplaced)
-    (property "Reference" "#PWR?" (id 0) (at 187.96 77.47 0)
+    (property "Reference" "#PWR0108" (id 0) (at 187.96 77.47 0)
       (effects (font (size 1.27 1.27)) hide)
     )
@@
       (effects (font (size 1.27 1.27)) (justify left))
     )
-    (property "Footprint" "Package_DIP:DIP-28_W15.24mm_LongPads" (id 2) (at 140.97 66.04 0)
+    (property "Footprint" "Socket:DIP_Socket-28_W11.9_W12.7_W15.24_W17.78_W18.5_3M_228-1277-00-0602J" (id 2) (at 140.97 66.04 0)
       (effects (font (size 1.27 1.27)) hide)
     )
@@
     )
     (path "/7f5bd2cb-38e8-4190-8121-88b1948fda1c"
-      (reference "#PWR?") (unit 1) (value "+5V") (footprint "")
+      (reference "#PWR0107") (unit 1) (value "+5V") (footprint "")
     )
     (path "/bda5a9a7-f2a6-4dac-9146-a85e15d84811"
-      (reference "#PWR?") (unit 1) (value "GND") (footprint "")
+      (reference "#PWR0108") (unit 1) (value "GND") (footprint "")
     )
     (path "/20c7b0cb-69cc-45e1-bc66-b0cdd6708f52"
@@
     )
     (path "/d1b9c1e5-14c1-4f12-b0cf-888fed203b23"
-      (reference "U1") (unit 1) (value "28C256") (footprint "Package_DIP:DIP-28_W15.24mm_LongPads")
-    )
-  )
+      (reference "U1") (unit 1) (value "28C256") (footprint "Socket:DIP_Socket-28_W11.9_W12.7_W15.24_W17.78_W18.5_3M_228-1277-00-0602J")
+    )
+  )
