File: memory/memory.kicad_pcb (KiCad board)
At the start: 2 copper layers, 76 x 84.1 mm, 6 parts, among them J1 Conn_01x02, J2 Conn_01x15, J3 Conn_01x08, J4 Conn_01x06, U1 28C256

Commit message: Memory board
Parts:
- U1: footprint Package_DIP:DIP-28_W15.24mm_LongPads -> Socket:DIP_Socket-28_W11.9_W12.7_W15.24_W17.78_W18.5_3M_228-1277-00-0602J
- moved C1 1.31 mm to (25.3, 31.7)
Connections:
- J4 pad 2: /a14 -> GND
- J4 pad 4: GND -> /a14
Routing:
- net /a9: track 90.2 -> 72.8 mm, vias 4 -> 2
- net /a14: track 87.2 -> 101.6 mm
- net /a10: track 101.9 -> 88.9 mm, vias 4 -> 2
- net /d7: track 148.3 -> 136.7 mm
- net /d6: track 143.2 -> 131.6 mm
- net /d4: track 133.1 -> 121.4 mm
- net /d3: track 128.0 -> 116.3 mm
- net /d5: track 138.1 -> 126.6 mm
- net /a11: track 80.5 -> 69.5 mm, vias 4 -> 2
- net /a8: track 87.2 -> 76.7 mm, vias 4 -> 2
- net /a13: track 56.1 -> 66.6 mm
- net +5V: track 119.3 -> 109.8 mm
- net /d1: track 76.7 -> 79.5 mm
- net /a12: track 34.3 -> 32.2 mm
- net Net-(J4-Pad1): track 15.2 -> 13.8 mm
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
Commit message: Fix: memory
Parts:
- moved C1 19.5 mm to (35.6, 48.3)
- moved J4 12.9 mm to (58.4, 89.3)
- moved U1 12.9 mm to (71.1, 66.4)
- moved J2 10.2 mm to (40.6, 27.2)
- moved J3 10.2 mm to (82.6, 27.2)
- moved J1 10.2 mm to (31.7, 27.2)
Routing:
- net /d2: track 80.3 -> 244.9 mm, vias 2 -> 4
- net /d1: track 79.5 -> 238.1 mm, vias 2 -> 4
- net /d0: track 78.1 -> 232.1 mm, vias 2 -> 4
- net /a14: track 101.6 -> 118.6 mm
- net /a7: track 34.3 -> 46.8 mm
- net /a5: track 34.3 -> 46.8 mm
- net /a0: track 34.3 -> 46.8 mm
- net /a4: track 34.3 -> 46.8 mm
- net /a3: track 34.3 -> 46.8 mm
- net /a2: track 34.3 -> 46.8 mm
- net /a1: track 34.3 -> 46.8 mm
- net /a6: track 34.4 -> 46.8 mm
- net /a9: track 72.8 -> 84.4 mm
- net /d3: track 116.3 -> 124.9 mm
- net GND: track 108.0 -> 116.3 mm
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Other:
- board size 76 x 84.1 mm -> 96.3 x 94.8 mm

Commit message: Backup
Parts:
- moved U1 16.3 mm to (81.3, 53.7)
- moved J4 13.5 mm to (67.3, 79.1)
- moved C1 7.27 mm to (35.6, 41.0)
Routing:
- net /d0: track 232.1 -> 76.6 mm, vias 4 -> 2
- net /d1: track 238.1 -> 94.6 mm, vias 4 -> 2
- net /d2: track 244.9 -> 105.7 mm, vias 4 -> 2
- net /a14: track 118.6 -> 70.8 mm, vias 2 -> 0
- net /d4: track 129.4 -> 92.6 mm
- net /d3: track 124.9 -> 92.6 mm
- net /a11: track 77.0 -> 106.8 mm
- net /d7: track 144.6 -> 116.7 mm, vias 2 -> 4
- net GND: track 116.3 -> 89.3 mm, vias 2 -> 0
- net /d6: track 139.5 -> 117.6 mm
- net /a9: track 84.4 -> 101.5 mm, vias 2 -> 4
- net /d5: track 134.6 -> 122.7 mm
- net /a12: track 40.2 -> 29.6 mm
- net +5V: track 117.8 -> 127.5 mm, vias 0 -> 2
- net /a10: track 96.7 -> 90.5 mm
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Other:
- board size 96.3 x 94.8 mm -> 98 x 62 mm
