File: top-layer/top-layer.kicad_pcb (KiCad board)
At the start: 2 copper layers, 76 x 127.3 mm, 19 parts, among them J1 Conn_01x02_Male, J2 Conn_01x15_Male, J3 Conn_01x08_Male, J4 Conn_01x05_Male, SW1 SW_Push, SW2 SW_Push, SW3 SW_Push, SW4 SW_Push, SW5 SW_Push, U2 W65C22SxP

Commit message: Fix: top layer
Parts:
- moved DS1 9.32 mm to (49.6, 88.9)
- moved R2 7.62 mm to (36.8, 127.0)
- moved SW1 7.62 mm to (39.9, 140.0)
- moved SW2 7.62 mm to (52.6, 140.0)
- moved SW3 7.62 mm to (65.3, 140.0)
- moved SW4 7.62 mm to (78.0, 140.0)
- moved SW5 7.62 mm to (90.7, 140.0)
- moved R1 7.62 mm to (36.8, 132.1)
- moved R3 7.62 mm to (54.6, 132.1)
- moved R4 7.62 mm to (72.4, 132.1)
- moved R5 7.62 mm to (90.2, 132.1)
- moved RV1 2.54 mm to (40.6, 78.7)
Routing:
- net +5V: track 304.3 -> 276.0 mm
- net GND: track 230.1 -> 246.7 mm
- net LCD_RS: track 31.2 -> 20.3 mm
- net /db1: track 28.5 -> 20.3 mm
- net /db7: track 28.5 -> 20.3 mm
- net /db2: track 28.5 -> 20.3 mm
- net /db6: track 28.5 -> 20.3 mm
- net /db4: track 28.5 -> 20.3 mm
- net LCD_RW: track 28.5 -> 20.3 mm
- net LCD_E: track 28.5 -> 20.3 mm
- net /db5: track 28.5 -> 20.3 mm
- net /db3: track 28.5 -> 20.3 mm
- net /db0: track 28.5 -> 20.3 mm
- net SW3: track 151.2 -> 143.6 mm
- net SW5: track 135.9 -> 128.3 mm
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Other:
- board size 76 x 127.3 mm -> 76 x 117.1 mm
