File: bus/bus.kicad_pcb (KiCad board)
At the start: 2 copper layers, 76 x 119.7 mm, 19 parts, among them J1 Conn_01x02, J10 Conn_01x02, J11 Conn_01x15, J12 Conn_01x08, J13 Conn_01x02, J14 Conn_01x15, J15 Conn_01x08, J16 Conn_01x05_Male, J2 Conn_01x15, J3 Conn_01x08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

Commit message: Fix: bus layout
Parts:
- moved J13 10.2 mm to (22.9, 129.5)
- moved J14 10.2 mm to (31.7, 129.5)
- moved J15 10.2 mm to (73.7, 129.5)
- moved J10 7.59 mm to (22.9, 111.8)
- moved J11 7.59 mm to (31.7, 111.8)
- moved J12 7.59 mm to (73.7, 111.8)
- moved J7 5.05 mm to (22.9, 94.0)
- moved J8 5.05 mm to (31.7, 94.0)
- moved J9 5.05 mm to (73.7, 94.0)
- moved J4 2.52 mm to (22.9, 76.2)
- moved J5 2.52 mm to (31.7, 76.2)
- moved J6 2.52 mm to (73.7, 76.2)
Routing:
- net VBUS: track 151.2 -> 141.1 mm
- net GND: track 147.7 -> 137.5 mm
- net D7: track 81.3 -> 71.1 mm
- net D6: track 81.3 -> 71.1 mm
- net D5: track 81.3 -> 71.1 mm
- net D4: track 81.3 -> 71.1 mm
- net D3: track 81.3 -> 71.1 mm
- net D2: track 81.3 -> 71.1 mm
- net D1: track 81.3 -> 71.1 mm
- net D0: track 81.3 -> 71.1 mm
- net A9: track 81.3 -> 71.1 mm
- net A8: track 81.3 -> 71.1 mm
- net A7: track 81.3 -> 71.1 mm
- net A6: track 81.3 -> 71.1 mm
- net A5: track 81.3 -> 71.1 mm
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Other:
- board size 76 x 119.7 mm -> 76 x 103 mm
Changed lines of the file:
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@@
   (setup
     (pad_to_mask_clearance 0)
+    (grid_origin 20.32 35.56)
     (pcbplotparams
       (layerselection 0x00010fc_ffffffff)
@@
   )
   (footprint "Connector_PinSocket_2.54mm:PinSocket_1x08_P2.54mm_Vertical" (layer "F.Cu")
-    (at 73.66 99.035 90)
+    (at 73.66 93.98 90)
     (descr "Through hole straight socket strip, 1x08, 2.54mm pitch, single row (from Kicad 4.0.7), script generated")
     (tags "Through hole socket strip THT 1x08 2.54mm single row")
@@
   )
   (footprint "Connector_PinSocket_2.54mm:PinSocket_1x15_P2.54mm_Vertical" (layer "F.Cu")
-    (at 31.74 99.035 90)
+    (at 31.74 93.98 90)
     (descr "Through hole straight socket strip, 1x15, 2.54mm pitch, single row (from Kicad 4.0.7), script generated")
     (tags "Through hole socket strip THT 1x15 2.54mm single row")
@@
   )
   (footprint "Connector_PinSocket_2.54mm:PinSocket_1x08_P2.54mm_Vertical" (layer "F.Cu")
-    (at 73.66 139.7 90)
+    (at 73.66 129.54 90)
     (descr "Through hole straight socket strip, 1x08, 2.54mm pitch, single row (from Kicad 4.0.7), script generated")
     (tags "Through hole socket strip THT 1x08 2.54mm single row")
@@
   )
   (footprint "Connector_PinSocket_2.54mm:PinSocket_1x15_P2.54mm_Vertical" (layer "F.Cu")
-    (at 31.74 119.355 90)
+    (at 31.74 111.76 90)
     (descr "Through hole straight socket strip, 1x15, 2.54mm pitch, single row (from Kicad 4.0.7), script generated")
     (tags "Through hole socket strip THT 1x15 2.54mm single row")
@@
   )
   (footprint "Connector_PinSocket_2.54mm:PinSocket_1x02_P2.54mm_Vertical" (layer "F.Cu")
-    (at 22.86 78.715 90)
+    (at 22.86 76.2 90)
     (descr "Through hole straight socket strip, 1x02, 2.54mm pitch, single row (from Kicad 4.0.7), script generated")
     (tags "Through hole socket strip THT 1x02 2.54mm single row")
@@
   )
   (footprint "Connector_PinSocket_2.54mm:PinSocket_1x15_P2.54mm_Vertical" (layer "F.Cu")
-    (at 31.74 139.7 90)
+    (at 31.74 129.54 90)
     (descr "Through hole straight socket strip, 1x15, 2.54mm pitch, single row (from Kicad 4.0.7), script generated")
     (tags "Through hole socket strip THT 1x15 2.54mm single row")
@@
   )
   (footprint "Connector_PinSocket_2.54mm:PinSocket_1x08_P2.54mm_Vertical" (layer "F.Cu")
-    (at 73.66 119.355 90)
+    (at 73.66 111.76 90)
     (descr "Through hole straight socket strip, 1x08, 2.54mm pitch, single row (from Kicad 4.0.7), script generated")
     (tags "Through hole socket strip THT 1x08 2.54mm single row")
@@
   )
   (footprint "Connector_PinSocket_2.54mm:PinSocket_1x08_P2.54mm_Vertical" (layer "F.Cu")
-    (at 73.66 78.715 90)
+    (at 73.66 76.2 90)
     (descr "Through hole straight socket strip, 1x08, 2.54mm pitch, single row (from Kicad 4.0.7), script generated")
     (tags "Through hole socket strip THT 1x08 2.54mm single row")
@@
   )
   (footprint "Connector_PinSocket_2.54mm:PinSocket_1x02_P2.54mm_Vertical" (layer "F.Cu")
-    (at 22.86 99.035 90)
+    (at 22.86 93.98 90)
     (descr "Through hole straight socket strip, 1x02, 2.54mm pitch, single row (from Kicad 4.0.7), script generated")
     (tags "Through hole socket strip THT 1x02 2.54mm single row")
@@
   )
   (footprint "Connector_PinSocket_2.54mm:PinSocket_1x15_P2.54mm_Vertical" (layer "F.Cu")
-    (at 31.74 78.715 90)
+    (at 31.74 76.2 90)
     (descr "Through hole straight socket strip, 1x15, 2.54mm pitch, single row (from Kicad 4.0.7), script generated")
     (tags "Through hole socket strip THT 1x15 2.54mm single row")
@@
   )
   (footprint "Connector_PinSocket_2.54mm:PinSocket_1x02_P2.54mm_Vertical" (layer "F.Cu")
-    (at 22.86 119.355 90)
+    (at 22.86 111.76 90)
     (descr "Through hole straight socket strip, 1x02, 2.54mm pitch, single row (from Kicad 4.0.7), script generated")
     (tags "Through hole socket strip THT 1x02 2.54mm single row")
@@
   )
   (footprint "Connector_PinSocket_2.54mm:PinSocket_1x02_P2.54mm_Vertical" (layer "F.Cu")
-    (at 22.86 139.7 90)
+    (at 22.86 129.54 90)
     (descr "Through hole straight socket strip, 1x02, 2.54mm pitch, single row (from Kicad 4.0.7), script generated")
     (tags "Through hole socket strip THT 1x02 2.54mm single row")
@@
     )
   )
-  (gr_rect (start 19.235 30.365) (end 95.235 150.025) (layer "Edge.Cuts") (width 0.1) (fill none))
+  (gr_rect (start 19.235 30.365) (end 95.235 133.365) (layer "Edge.Cuts") (width 0.1) (fill none))
   (segment (start 50.8 40.64) (end 54.61 40.64) (width 1.5) (layer "B.Cu") (net 1))
   (segment (start 54.61 40.64) (end 60.96 34.29) (width 1.5) (layer "B.Cu") (net 1))
   (segment (start 48.26 43.18) (end 48.26 40.64) (width 1.5) (layer "B.Cu") (net 2))
+  (segment (start 22.86 58.42) (end 22.86 129.54) (width 1.5) (layer "B.Cu") (net 2))
   (segment (start 73.66 43.1) (end 73.66 45.72) (width 1.5) (layer "B.Cu") (net 2))
   (segment (start 68.58 48.26) (end 63.5 43.18) (width 1.5) (layer "B.Cu") (net 2))
@@
   (segment (start 38.29 40.64) (end 48.26 40.64) (width 1.5) (layer "B.Cu") (net 2))
   (segment (start 55.88 45.72) (end 50.8 45.72) (width 1.5) (layer "B.Cu") (net 2))
-  (segment (start 22.86 58.42) (end 22.86 139.7) (width 1.5) (layer "B.Cu") (net 2))
   (segment (start 63.5 43.18) (end 58.42 43.18) (width 1.5) (layer "B.Cu") (net 2))
   (segment (start 58.42 43.18) (end 55.88 45.72) (width 1.5) (layer "B.Cu") (net 2))
@@
   (segment (start 73.66 53.34) (end 67.31 53.34) (width 1.5) (layer "B.Cu") (net 3))
   (segment (start 67.31 53.34) (end 60.96 46.99) (width 1.5) (layer "B.Cu") (net 3))
-  (segment (start 25.4 58.42) (end 25.4 139.7) (width 1.5) (layer "B.Cu") (net 3))
   (segment (start 60.96 46.99) (end 57.15 50.8) (width 1.5) (layer "B.Cu") (net 3))
-  (segment (start 31.74 58.42) (end 31.74 139.7) (width 1.5) (layer "B.Cu") (net 4))
-  (segment (start 34.28 139.7) (end 34.28 58.42) (width 1.5) (layer "B.Cu") (net 5))
-  (segment (start 36.82 58.42) (end 36.82 139.7) (width 1.5) (layer "B.Cu") (net 6))
-  (segment (start 39.36 139.7) (end 39.36 58.42) (width 1.5) (layer "B.Cu") (net 7))
-  (segment (start 41.9 58.42) (end 41.9 139.7) (width 1.5) (layer "B.Cu") (net 8))
-  (segment (start 44.44 139.7) (end 44.44 58.42) (width 1.5) (layer "B.Cu") (net 9))
-  (segment (start 46.98 58.42) (end 46.98 139.7) (width 1.5) (layer "B.Cu") (net 10))
-  (segment (start 49.52 139.7) (end 49.52 58.42) (width 1.5) (layer "B.Cu") (net 11))
-  (segment (start 52.06 58.42) (end 52.06 139.7) (width 1.5) (layer "B.Cu") (net 12))
-  (segment (start 54.6 139.7) (end 54.6 58.42) (width 1.5) (layer "B.Cu") (net 13))
-  (segment (start 57.14 58.42) (end 57.14 139.7) (width 1.5) (layer "B.Cu") (net 14))
-  (segment (start 59.68 139.7) (end 59.68 58.42) (width 1.5) (layer "B.Cu") (net 15))
-  (segment (start 62.22 58.42) (end 62.22 139.7) (width 1.5) (layer "B.Cu") (net 16))
-  (segment (start 64.76 139.7) (end 64.76 58.42) (width 1.5) (layer "B.Cu") (net 17))
-  (segment (start 67.3 58.42) (end 67.3 139.7) (width 1.5) (layer "B.Cu") (net 18))
-  (segment (start 73.66 58.42) (end 73.66 139.7) (width 1.5) (layer "B.Cu") (net 19))
-  (segment (start 76.2 139.7) (end 76.2 58.42) (width 1.5) (layer "B.Cu") (net 20))
-  (segment (start 78.74 58.42) (end 78.74 139.7) (width 1.5) (layer "B.Cu") (net 21))
-  (segment (start 81.28 58.42) (end 81.28 139.7) (width 1.5) (layer "B.Cu") (net 22))
-  (segment (start 83.82 139.7) (end 83.82 58.42) (width 1.5) (layer "B.Cu") (net 23))
-  (segment (start 86.36 58.42) (end 86.36 139.7) (width 1.5) (layer "B.Cu") (net 24))
-  (segment (start 88.9 139.7) (end 88.9 58.42) (width 1.5) (layer "B.Cu") (net 25))
-  (segment (start 91.44 58.42) (end 91.44 139.7) (width 1.5) (layer "B.Cu") (net 26))
+  (segment (start 25.4 58.42) (end 25.4 129.54) (width 1.5) (layer "B.Cu") (net 3))
+  (segment (start 31.74 58.42) (end 31.74 129.54) (width 1.5) (layer "B.Cu") (net 4))
+  (segment (start 34.28 129.54) (end 34.28 58.42) (width 1.5) (layer "B.Cu") (net 5))
+  (segment (start 36.82 58.42) (end 36.82 129.54) (width 1.5) (layer "B.Cu") (net 6))
+  (segment (start 39.36 58.42) (end 39.36 129.54) (width 1.5) (layer "B.Cu") (net 7))
+  (segment (start 41.9 58.42) (end 41.9 129.54) (width 1.5) (layer "B.Cu") (net 8))
+  (segment (start 44.44 129.54) (end 44.44 58.42) (width 1.5) (layer "B.Cu") (net 9))
+  (segment (start 46.98 58.42) (end 46.98 129.54) (width 1.5) (layer "B.Cu") (net 10))
+  (segment (start 49.52 129.54) (end 49.52 58.42) (width 1.5) (layer "B.Cu") (net 11))
+  (segment (start 52.06 58.42) (end 52.06 129.54) (width 1.5) (layer "B.Cu") (net 12))
+  (segment (start 54.6 129.54) (end 54.6 58.42) (width 1.5) (layer "B.Cu") (net 13))
+  (segment (start 57.14 58.42) (end 57.14 129.54) (width 1.5) (layer "B.Cu") (net 14))
+  (segment (start 59.68 129.54) (end 59.68 58.42) (width 1.5) (layer "B.Cu") (net 15))
+  (segment (start 62.22 58.42) (end 62.22 129.54) (width 1.5) (layer "B.Cu") (net 16))
+  (segment (start 64.76 129.54) (end 64.76 58.42) (width 1.5) (layer "B.Cu") (net 17))
+  (segment (start 67.3 58.42) (end 67.3 129.54) (width 1.5) (layer "B.Cu") (net 18))
+  (segment (start 73.66 58.42) (end 73.66 129.54) (width 1.5) (layer "B.Cu") (net 19))
+  (segment (start 76.2 129.54) (end 76.2 58.42) (width 1.5) (layer "B.Cu") (net 20))
+  (segment (start 78.74 58.42) (end 78.74 129.54) (width 1.5) (layer "B.Cu") (net 21))
+  (segment (start 81.28 58.42) (end 81.28 129.54) (width 1.5) (layer "B.Cu") (net 22))
+  (segment (start 83.82 129.54) (end 83.82 58.42) (width 1.5) (layer "B.Cu") (net 23))
+  (segment (start 86.36 58.42) (end 86.36 129.54) (width 1.5) (layer "B.Cu") (net 24))
+  (segment (start 88.9 129.54) (end 88.9 58.42) (width 1.5) (layer "B.Cu") (net 25))
+  (segment (start 91.44 58.42) (end 91.44 129.54) (width 1.5) (layer "B.Cu") (net 26))
   (segment (start 74.859022 40.6) (end 79.899022 35.56) (width 1.5) (layer "B.Cu") (net 27))
   (segment (start 73.66 40.6) (end 74.859022 40.6) (width 1.5) (layer "B.Cu") (net 27))
