File: cpu/cpu.kicad_sch (KiCad schematic)
At the start: 7 parts, among them J1 Conn_01x02, J2 Conn_01x15, J3 Conn_01x08, J4 Conn_01x02_Male, U1 W65C02SxP

Commit message: WIP: cpu
Parts:
- removed J4: Conn_01x02_Male, Connector_PinHeader_2.54mm:PinHeader_1x02_P2.54mm_Vertical, symbol Connector:Conn_01x02_Male
- added C10, C2, C6: 0.1uF, Capacitor_THT:C_Disc_D6.0mm_W2.5mm_P5.00mm, symbol Device:C
- added C3: 10uF, Capacitor_THT:CP_Radial_D5.0mm_P2.50mm, symbol Device:C_Polarized
- added C4, C9: .01uF, Capacitor_THT:C_Rect_L7.0mm_W2.5mm_P5.00mm, symbol Device:C
- added C5: .1uF, Capacitor_THT:C_Rect_L7.0mm_W2.5mm_P5.00mm, symbol Device:C
- added C7: 30pF, Capacitor_THT:C_Disc_D3.0mm_W1.6mm_P2.50mm, symbol Device:C
- added C8: 3pF, Capacitor_THT:C_Disc_D3.0mm_W1.6mm_P2.50mm, symbol Device:C
- added J4, J7: Conn_01x01_Male, symbol Connector:Conn_01x01_Male
- added J5, J8: Conn_01x03_Male, symbol Connector:Conn_01x03_Male
- added J6: Conn_01x02_Male, symbol Connector:Conn_01x02_Male
- added R2: 47K, Resistor_THT:R_Axial_DIN0411_L9.9mm_D3.6mm_P12.70mm_Horizontal, symbol Device:R
- added R3: 1M, Resistor_THT:R_Axial_DIN0411_L9.9mm_D3.6mm_P12.70mm_Horizontal, symbol Device:R
- added R4, R5: 10M, Resistor_THT:R_Axial_DIN0207_L6.3mm_D2.5mm_P10.16mm_Horizontal, symbol Device:R
- added SW1: SW_Push, symbol Switch:SW_Push
- added U2: 74HC00, symbol 74xx:74HC00
- added U3: NE555P, Package_DIP:DIP-8_W7.62mm, symbol Timer:NE555P
- added U4: 74HC14, symbol 74xx:74HC14
- added Y1: Crystal, Crystal:Crystal_C26-LF_D2.1mm_L6.5mm_Vertical, symbol Device:Crystal
Connections:
- net +5V: now also C10.2, C2.2, C6.2, R2.2, R3.2, U2.14 (VCC), U3.4 (R), U3.8 (VCC), U4.14 (VCC)
- net A15: now also U2.1, U2.2
- net CLOCK_IN_PIN: now also C9.1, U4.4
- net CLOCK_OUT_PIN: now also J6.1 (Pin_1), J6.2 (Pin_2), U2.4
- net CS_6522_PIN: now also J5.1 (Pin_1), U2.8
- net CS_MEMORY_PIN: now also J5.3 (Pin_3), U2.6
- net CS_PROGRAM_PIN: now also J5.2 (Pin_2), U2.10, U2.3, U2.5
- net GND: now also C10.1, C2.1, C3.2, C4.2, C5.2, C6.1, C7.1, C8.1, C9.2, SW1.1, U2.7 (GND), U3.1 (GND), U4.7 (GND)
- net RESET_PIN: now also J7.1 (Pin_1), U2.11
- net 6502_RW: now reaches U1.34 (R/~{W})
- net 6502_RW: now also J8.1 (Pin_1), J8.2 (Pin_2), J8.3 (Pin_3)
- net IRQ_PIN renamed 6502_IRQ
- net 6502_IRQ: now also J4.1 (Pin_1)
- net a0: no longer names the net of J2.1 (Pin_1)
- net a1: no longer names the net of J2.2 (Pin_2)
- net a10: no longer names the net of J2.11 (Pin_11)
- net a11: no longer names the net of J2.12 (Pin_12)
- net a12: no longer names the net of J2.13 (Pin_13)
- net a13: no longer names the net of J2.14 (Pin_14)
- net a14 renamed A14
- net A14: now also U2.9
- net a2: no longer names the net of J2.3 (Pin_3)
- net a3: no longer names the net of J2.4 (Pin_4)
- net a4: no longer names the net of J2.5 (Pin_5)
- net a5: no longer names the net of J2.6 (Pin_6)
- net a6: no longer names the net of J2.7 (Pin_7)
- net a7: no longer names the net of J2.8 (Pin_8)
- net a8: no longer names the net of J2.9 (Pin_9)
- net a9: no longer names the net of J2.10 (Pin_10)
- net d0: no longer names the net of J3.1 (Pin_1)
- net d1: no longer names the net of J3.2 (Pin_2)
- net d2: no longer names the net of J3.3 (Pin_3)
- net d3: no longer names the net of J3.4 (Pin_4)
- net d4: no longer names the net of J3.5 (Pin_5)
- net d5: no longer names the net of J3.6 (Pin_6)
- net d6: no longer names the net of J3.7 (Pin_7)
- net d7: no longer names the net of J3.8 (Pin_8)
- new net: C7.2, R4.1, U4.1, Y1.1
- new net: R4.2, R5.1, U4.2, U4.3
- new net: C5.1, R3.1, SW1.2, U3.2 (TR)
- new net: U2.12, U2.13, U3.3 (Q)
- new net: C4.1, U3.5 (CV)
- new net: C3.1, R2.1, U3.6 (THR), U3.7 (DIS)
- new net: C8.2, R5.2, Y1.2
Other:
- moved on the sheet: C1, J1

Commit message: cpu: before routing
Parts:
- J4, J7: footprint (none) -> Connector_PinHeader_2.54mm:PinHeader_1x01_P2.54mm_Vertical
- J5, J8: footprint (none) -> Connector_PinHeader_2.54mm:PinHeader_1x03_P2.54mm_Vertical
- J6: footprint (none) -> Connector_PinHeader_2.54mm:PinHeader_1x02_P2.54mm_Vertical
- R5: value 10M -> 270K
- SW1: footprint (none) -> Button_Switch_THT:SW_PUSH_6mm
- U1: footprint (none) -> Package_DIP:DIP-40_W15.24mm_Socket_LongPads
- U2, U4: footprint (none) -> Package_DIP:DIP-14_W7.62mm_Socket_LongPads
Changed lines of the file:
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@@
     (property "Reference" "J8" (id 0) (at 254.635 60.96 0))
     (property "Value" "Conn_01x03_Male" (id 1) (at 254.635 63.5 0))
-    (property "Footprint" "" (id 2) (at 254 68.58 0)
+    (property "Footprint" "Connector_PinHeader_2.54mm:PinHeader_1x03_P2.54mm_Vertical" (id 2) (at 254 68.58 0)
       (effects (font (size 1.27 1.27)) hide)
     )
@@
     (property "Reference" "U4" (id 0) (at 207.01 90.17 0))
     (property "Value" "74HC14" (id 1) (at 207.01 92.71 0))
-    (property "Footprint" "" (id 2) (at 207.01 99.06 0)
+    (property "Footprint" "Package_DIP:DIP-14_W7.62mm_Socket_LongPads" (id 2) (at 207.01 99.06 0)
       (effects (font (size 1.27 1.27)) hide)
     )
@@
     (property "Reference" "U2" (id 0) (at 129.54 177.8 0))
     (property "Value" "74HC00" (id 1) (at 129.54 180.34 0))
-    (property "Footprint" "" (id 2) (at 129.54 186.69 0)
+    (property "Footprint" "Package_DIP:DIP-14_W7.62mm_Socket_LongPads" (id 2) (at 129.54 186.69 0)
       (effects (font (size 1.27 1.27)) hide)
     )
@@
     (property "Reference" "U4" (id 0) (at 234.95 90.17 0))
     (property "Value" "74HC14" (id 1) (at 234.95 92.71 0))
-    (property "Footprint" "" (id 2) (at 234.95 99.06 0)
+    (property "Footprint" "Package_DIP:DIP-14_W7.62mm_Socket_LongPads" (id 2) (at 234.95 99.06 0)
       (effects (font (size 1.27 1.27)) hide)
     )
@@
     (property "Reference" "U2" (id 0) (at 86.36 24.13 0))
     (property "Value" "74HC00" (id 1) (at 86.36 26.67 0))
-    (property "Footprint" "" (id 2) (at 86.36 33.02 0)
+    (property "Footprint" "Package_DIP:DIP-14_W7.62mm_Socket_LongPads" (id 2) (at 86.36 33.02 0)
       (effects (font (size 1.27 1.27)) hide)
     )
@@
     (property "Reference" "J4" (id 0) (at 250.825 15.24 0))
     (property "Value" "Conn_01x01_Male" (id 1) (at 250.825 17.78 0))
-    (property "Footprint" "" (id 2) (at 250.19 20.32 0)
+    (property "Footprint" "Connector_PinHeader_2.54mm:PinHeader_1x01_P2.54mm_Vertical" (id 2) (at 250.19 20.32 0)
       (effects (font (size 1.27 1.27)) hide)
     )
@@
       (effects (font (size 1.27 1.27)) (justify left))
     )
-    (property "Footprint" "" (id 2) (at 36.83 144.78 0)
+    (property "Footprint" "Package_DIP:DIP-14_W7.62mm_Socket_LongPads" (id 2) (at 36.83 144.78 0)
       (effects (font (size 1.27 1.27)) hide)
     )
@@
   )
   (symbol (lib_id "65xx:W65C02SxP") (at 151.13 67.31 0) (unit 1)
-    (in_bom yes) (on_board yes) (fields_autoplaced)
+    (in_bom yes) (on_board yes)
     (property "Reference" "U1" (id 0) (at 153.1494 27.94 0)
       (effects (font (size 1.27 1.27)) (justify left))
     )
-    (property "Value" "W65C02SxP" (id 1) (at 153.1494 30.48 0)
+    (property "Value" "W65C02SxP" (id 1) (at 152.4 30.48 0)
       (effects (font (size 1.27 1.27) bold italic) (justify left))
     )
-    (property "Footprint" "" (id 2) (at 151.13 16.51 0)
+    (property "Footprint" "Package_DIP:DIP-40_W15.24mm_Socket_LongPads" (id 2) (at 151.13 16.51 0)
       (effects (font (size 1.27 1.27)) hide)
     )
@@
     (property "Reference" "U2" (id 0) (at 90.17 173.99 0))
     (property "Value" "74HC00" (id 1) (at 90.17 176.53 0))
-    (property "Footprint" "" (id 2) (at 90.17 182.88 0)
+    (property "Footprint" "Package_DIP:DIP-14_W7.62mm_Socket_LongPads" (id 2) (at 90.17 182.88 0)
       (effects (font (size 1.27 1.27)) hide)
     )
@@
     (property "Reference" "J7" (id 0) (at 254.635 52.07 0))
     (property "Value" "Conn_01x01_Male" (id 1) (at 254.635 54.61 0))
-    (property "Footprint" "" (id 2) (at 254 57.15 0)
+    (property "Footprint" "Connector_PinHeader_2.54mm:PinHeader_1x01_P2.54mm_Vertical" (id 2) (at 254 57.15 0)
       (effects (font (size 1.27 1.27)) hide)
     )
@@
     (property "Reference" "J6" (id 0) (at 254.635 39.37 0))
     (property "Value" "Conn_01x02_Male" (id 1) (at 254.635 41.91 0))
-    (property "Footprint" "" (id 2) (at 254 44.45 0)
+    (property "Footprint" "Connector_PinHeader_2.54mm:PinHeader_1x02_P2.54mm_Vertical" (id 2) (at 254 44.45 0)
       (effects (font (size 1.27 1.27)) hide)
     )
@@
     (property "Reference" "J5" (id 0) (at 250.825 24.13 0))
     (property "Value" "Conn_01x03_Male" (id 1) (at 250.825 26.67 0))
-    (property "Footprint" "" (id 2) (at 250.19 31.75 0)
+    (property "Footprint" "Connector_PinHeader_2.54mm:PinHeader_1x03_P2.54mm_Vertical" (id 2) (at 250.19 31.75 0)
       (effects (font (size 1.27 1.27)) hide)
     )
@@
     (property "Reference" "SW1" (id 0) (at 20.32 26.67 0))
     (property "Value" "SW_Push" (id 1) (at 20.32 29.21 0))
-    (property "Footprint" "" (id 2) (at 20.32 29.21 0)
+    (property "Footprint" "Button_Switch_THT:SW_PUSH_6mm" (id 2) (at 20.32 29.21 0)
       (effects (font (size 1.27 1.27)) hide)
     )
@@
       (effects (font (size 1.27 1.27)) (justify left))
     )
-    (property "Footprint" "" (id 2) (at 274.32 144.78 0)
+    (property "Footprint" "Package_DIP:DIP-14_W7.62mm_Socket_LongPads" (id 2) (at 274.32 144.78 0)
       (effects (font (size 1.27 1.27)) hide)
     )
@@
     (property "Reference" "U2" (id 0) (at 43.18 176.53 0))
     (property "Value" "74HC00" (id 1) (at 43.18 179.07 0))
-    (property "Footprint" "" (id 2) (at 43.18 185.42 0)
+    (property "Footprint" "Package_DIP:DIP-14_W7.62mm_Socket_LongPads" (id 2) (at 43.18 185.42 0)
       (effects (font (size 1.27 1.27)) hide)
     )
@@
       (effects (font (size 1.27 1.27)) (justify left))
     )
-    (property "Value" "10M" (id 1) (at 217.17 105.4099 0)
+    (property "Value" "270K" (id 1) (at 217.17 105.4099 0)
       (effects (font (size 1.27 1.27)) (justify left))
     )
@@
     )
     (path "/58f2669f-fc2d-4ea9-bd6c-ddb25e1d626e"
-      (reference "J4") (unit 1) (value "Conn_01x01_Male") (footprint "")
+      (reference "J4") (unit 1) (value "Conn_01x01_Male") (footprint "Connector_PinHeader_2.54mm:PinHeader_1x01_P2.54mm_Vertical")
     )
     (path "/9d91386f-505d-45f5-9efe-0e911ed1e521"
-      (reference "J5") (unit 1) (value "Conn_01x03_Male") (footprint "")
+      (reference "J5") (unit 1) (value "Conn_01x03_Male") (footprint "Connector_PinHeader_2.54mm:PinHeader_1x03_P2.54mm_Vertical")
     )
     (path "/9be83551-1969-4198-8d13-104f87f594ec"
-      (reference "J6") (unit 1) (value "Conn_01x02_Male") (footprint "")
+      (reference "J6") (unit 1) (value "Conn_01x02_Male") (footprint "Connector_PinHeader_2.54mm:PinHeader_1x02_P2.54mm_Vertical")
     )
     (path "/8f4db84f-8648-4055-914d-a3395163e1d3"
-      (reference "J7") (unit 1) (value "Conn_01x01_Male") (footprint "")
+      (reference "J7") (unit 1) (value "Conn_01x01_Male") (footprint "Connector_PinHeader_2.54mm:PinHeader_1x01_P2.54mm_Vertical")
     )
     (path "/0139d8d7-e5f7-4566-a189-2a0c55a8f3a8"
-      (reference "J8") (unit 1) (value "Conn_01x03_Male") (footprint "")
+      (reference "J8") (unit 1) (value "Conn_01x03_Male") (footprint "Connector_PinHeader_2.54mm:PinHeader_1x03_P2.54mm_Vertical")
     )
     (path "/c63f3192-7de6-4e2a-bb43-77731d75c0ed"
@@
     )
     (path "/f03a9c39-5f19-414b-a28a-5f4bae37f172"
-      (reference "R5") (unit 1) (value "10M") (footprint "Resistor_THT:R_Axial_DIN0207_L6.3mm_D2.5mm_P10.16mm_Horizontal")
+      (reference "R5") (unit 1) (value "270K") (footprint "Resistor_THT:R_Axial_DIN0207_L6.3mm_D2.5mm_P10.16mm_Horizontal")
     )
     (path "/af71175c-f1c6-4dc1-b188-d9d7ed8bf11d"
-      (reference "SW1") (unit 1) (value "SW_Push") (footprint "")
+      (reference "SW1") (unit 1) (value "SW_Push") (footprint "Button_Switch_THT:SW_PUSH_6mm")
     )
     (path "/7523562a-efe0-4507-ad96-7570739c8920"
-      (reference "U1") (unit 1) (value "W65C02SxP") (footprint "")
+      (reference "U1") (unit 1) (value "W65C02SxP") (footprint "Package_DIP:DIP-40_W15.24mm_Socket_LongPads")
     )
     (path "/d17c02e1-8f03-44cd-a18c-77e78719dce4"
-      (reference "U2") (unit 1) (value "74HC00") (footprint "")
+      (reference "U2") (unit 1) (value "74HC00") (footprint "Package_DIP:DIP-14_W7.62mm_Socket_LongPads")
     )
     (path "/7fa8a569-0450-4b0c-984a-257661b17cdb"
-      (reference "U2") (unit 2) (value "74HC00") (footprint "")
+      (reference "U2") (unit 2) (value "74HC00") (footprint "Package_DIP:DIP-14_W7.62mm_Socket_LongPads")
     )
     (path "/2ce15560-87e2-4227-ac08-0adeae2f86f4"
-      (reference "U2") (unit 3) (value "74HC00") (footprint "")
+      (reference "U2") (unit 3) (value "74HC00") (footprint "Package_DIP:DIP-14_W7.62mm_Socket_LongPads")
     )
     (path "/45f7480b-0109-4fe0-b0ce-0a57dc54c1ff"
-      (reference "U2") (unit 4) (value "74HC00") (footprint "")
+      (reference "U2") (unit 4) (value "74HC00") (footprint "Package_DIP:DIP-14_W7.62mm_Socket_LongPads")
     )
     (path "/630dd454-b3d7-426f-a6d8-1bfb27bd1710"
-      (reference "U2") (unit 5) (value "74HC00") (footprint "")
+      (reference "U2") (unit 5) (value "74HC00") (footprint "Package_DIP:DIP-14_W7.62mm_Socket_LongPads")
     )
     (path "/235ee765-527b-4fc1-8b80-734c41d1c6b2"
@@
     )
     (path "/14485727-abbd-4b43-8f1f-a8c78970c408"
-      (reference "U4") (unit 1) (value "74HC14") (footprint "")
+      (reference "U4") (unit 1) (value "74HC14") (footprint "Package_DIP:DIP-14_W7.62mm_Socket_LongPads")
     )
     (path "/35d37778-2115-4681-879c-996be88dc8d6"
-      (reference "U4") (unit 2) (value "74HC14") (footprint "")
+      (reference "U4") (unit 2) (value "74HC14") (footprint "Package_DIP:DIP-14_W7.62mm_Socket_LongPads")
     )
     (path "/b38f5484-f73c-452c-b7b9-7277f657af65"
-      (reference "U4") (unit 7) (value "74HC14") (footprint "")
+      (reference "U4") (unit 7) (value "74HC14") (footprint "Package_DIP:DIP-14_W7.62mm_Socket_LongPads")
     )
     (path "/8defaec3-fd2b-4f84-a861-10797c9636b8"

Commit message: CPU done
Parts:
- added unit 6 of U4
- added unit 4 of U4
- added unit 5 of U4
- added unit 3 of U4
Connections:
- net CS_6522_PIN: now also J5.3 (Pin_3); no longer J5.1 (Pin_1)
- net CS_MEMORY_PIN: now also J5.2 (Pin_2); no longer J5.3 (Pin_3)
- net CS_PROGRAM_PIN: now also J5.1 (Pin_1); no longer J5.2 (Pin_2)
- net GND: now also U4.11, U4.13, U4.5, U4.9
- net CLOCK_INV: now reaches U2.12, U2.13, U3.3 (Q)
- net a1: now reaches U1.10 (A1)
- net a2: now reaches U1.11 (A2)
- net a3: now reaches U1.12 (A3)
- net a4: now reaches U1.13 (A4)
- net a5: now reaches U1.14 (A5)
- net a6: now reaches U1.15 (A6)
- net a7: now reaches U1.16 (A7)
- net a8: now reaches U1.17 (A8)
- net a9: now reaches U1.18 (A9)
- net a10: now reaches U1.19 (A10)
- net a11: now reaches U1.20 (A11)
- net a12: now reaches U1.22 (A12)
- net a13: now reaches U1.23 (A13)
- net d7: now reaches U1.26 (D7)
- net d6: now reaches U1.27 (D6)
- net d5: now reaches U1.28 (D5)
- net d4: now reaches U1.29 (D4)
- net d3: now reaches U1.30 (D3)
- net d2: now reaches U1.31 (D2)
- net d1: now reaches U1.32 (D1)
- net d0: now reaches U1.33 (D0)
- net a0: now reaches U1.9 (A0)
- no-connect marks 5 -> 9

Commit message: Fix: cpu
Parts:
- added J9: Conn_01x02_Male, Connector_PinHeader_2.54mm:PinHeader_1x02_P2.54mm_Vertical, symbol Connector:Conn_01x02_Male
Connections:
- net CLOCK_IN_PIN: now also J9.1 (Pin_1); no longer U1.37 (ϕ0)
- new net: J9.2 (Pin_2), U1.37 (ϕ0)
Changed lines of the file:
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@@
+    (stroke (width 0) (type default) (color 0 0 0 0))
+  )
+  (wire (pts (xy 113.03 44.45) (xy 135.89 44.45))
     (stroke (width 0) (type default) (color 0 0 0 0))
   )
@@
     (stroke (width 0) (type default) (color 0 0 0 0))
   )
+  (wire (pts (xy 113.03 41.91) (xy 118.11 41.91))
+    (stroke (width 0) (type default) (color 0 0 0 0))
+  )
   (wire (pts (xy 274.32 130.81) (xy 274.32 132.08))
     (stroke (width 0) (type default) (color 0 0 0 0))
@@
   )
   (wire (pts (xy 41.91 44.45) (xy 39.37 44.45))
-    (stroke (width 0) (type default) (color 0 0 0 0))
-  )
-  (wire (pts (xy 133.35 44.45) (xy 135.89 44.45))
     (stroke (width 0) (type default) (color 0 0 0 0))
   )
@@
     )
   )
-  (global_label "CLOCK_IN_PIN" (shape input) (at 133.35 44.45 180) (fields_autoplaced)
-    (effects (font (size 1.27 1.27)) (justify right))
-    (property "Intersheet References" "${INTERSHEET_REFS}" (id 0) (at 117.6926 44.3706 0)
-      (effects (font (size 1.27 1.27)) (justify right) hide)
+  (global_label "CLOCK_IN_PIN" (shape input) (at 118.11 41.91 0) (fields_autoplaced)
+    (effects (font (size 1.27 1.27)) (justify left))
+    (property "Intersheet References" "${INTERSHEET_REFS}" (id 0) (at 133.7674 41.9894 0)
+      (effects (font (size 1.27 1.27)) (justify left) hide)
     )
   )
@@
     )
     (pin "1")
+  )
+  (symbol (lib_id "Connector:Conn_01x02_Male") (at 107.95 41.91 0) (unit 1)
+    (in_bom yes) (on_board yes) (fields_autoplaced)
+    (property "Reference" "J9" (id 0) (at 108.585 36.83 0))
+    (property "Value" "Conn_01x02_Male" (id 1) (at 108.585 39.37 0))
+    (property "Footprint" "Connector_PinHeader_2.54mm:PinHeader_1x02_P2.54mm_Vertical" (id 2) (at 107.95 41.91 0)
+      (effects (font (size 1.27 1.27)) hide)
+    )
+    (property "Datasheet" "~" (id 3) (at 107.95 41.91 0)
+      (effects (font (size 1.27 1.27)) hide)
+    )
+    (pin "1")
+    (pin "2")
   )
   (symbol (lib_id "65xx:W65C02SxP") (at 151.13 67.31 0) (unit 1)
@@
       (reference "J8") (unit 1) (value "Conn_01x03_Male") (footprint "Connector_PinHeader_2.54mm:PinHeader_1x03_P2.54mm_Vertical")
     )
+    (path "/72a650f3-0b2b-4088-8c36-c13d3bf3d1f7"
+      (reference "J9") (unit 1) (value "Conn_01x02_Male") (footprint "Connector_PinHeader_2.54mm:PinHeader_1x02_P2.54mm_Vertical")
+    )
     (path "/c63f3192-7de6-4e2a-bb43-77731d75c0ed"
