File: cpu/cpu.kicad_pcb (KiCad board)
At the start: 2 copper layers, 76 x 119.7 mm, 29 parts, among them J1 Conn_01x02, J2 Conn_01x15, J3 Conn_01x08, J4 Conn_01x01_Male, J5 Conn_01x03_Male, J6 Conn_01x02_Male, J7 Conn_01x01_Male, J8 Conn_01x03_Male, SW1 SW_Push, U1 W65C02SxP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

Commit message: CPU done
Parts:
- moved C4 147.3 mm to (54.6, 109.2)
- moved C10 145.7 mm to (49.5, 94.0)
- moved R3 144.8 mm to (30.5, 109.2)
- moved C5 144.5 mm to (26.7, 102.8), turned to 90 degrees
- moved R2 143.5 mm to (62.2, 108.0)
- moved SW1 139.2 mm to (32.9, 97.8)
- moved U3 138.7 mm to (48.3, 97.8)
- moved C3 122.3 mm to (67.3, 99.1), turned to 0 degrees
- moved J5 90.5 mm to (116.8, 91.4)
- moved U2 88.4 mm to (105.4, 81.3)
- moved C9 66.7 mm to (99.2, 119.4), turned to -90 degrees
- moved C8 62.9 mm to (83.9, 111.8), turned to 90 degrees
- moved C6 61.5 mm to (116.9, 114.3), turned to 90 degrees
- moved U4 59.6 mm to (105.5, 109.3)
- moved J6 58.0 mm to (111.8, 48.3), turned to 0 degrees
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Connections:
- net Net-(J2-Pad1) renamed /a0
- net Net-(J2-Pad10) renamed /a9
- net Net-(J2-Pad11) renamed /a10
- net Net-(J2-Pad12) renamed /a11
- net Net-(J2-Pad13) renamed /a12
- net Net-(J2-Pad14) renamed /a13
- net Net-(J2-Pad2) renamed /a1
- net Net-(J2-Pad3) renamed /a2
- net Net-(J2-Pad4) renamed /a3
- net Net-(J2-Pad5) renamed /a4
- net Net-(J2-Pad6) renamed /a5
- net Net-(J2-Pad7) renamed /a6
- net Net-(J2-Pad8) renamed /a7
- net Net-(J2-Pad9) renamed /a8
- net Net-(J3-Pad1) renamed /d0
- net Net-(J3-Pad2) renamed /d1
- net Net-(J3-Pad3) renamed /d2
- net Net-(J3-Pad4) renamed /d3
- net Net-(J3-Pad5) renamed /d4
- net Net-(J3-Pad6) renamed /d5
- net Net-(J3-Pad7) renamed /d6
- net Net-(J3-Pad8) renamed /d7
- net Net-(U2-Pad12) renamed /CLOCK_INV
- J5 pad 1: CS_6522_PIN -> CS_PROGRAM_PIN
- J5 pad 2: CS_PROGRAM_PIN -> CS_MEMORY_PIN
- J5 pad 3: CS_MEMORY_PIN -> CS_6522_PIN
- U4 pad 10: (no net) -> unconnected-(U4-Pad10)
- U4 pad 11: (no net) -> GND
- U4 pad 12: (no net) -> unconnected-(U4-Pad12)
- U4 pad 13: (no net) -> GND
- U4 pad 5: (no net) -> GND
- U4 pad 6: (no net) -> unconnected-(U4-Pad6)
- U4 pad 8: (no net) -> unconnected-(U4-Pad8)
- U4 pad 9: (no net) -> GND
Routing:
- net GND: track 0.00 -> 320.4 mm, vias 0 -> 6
- net +5V: track 0.00 -> 300.4 mm, vias 0 -> 10
- net /a11: track 0.00 -> 171.6 mm, vias 0 -> 2
- net /a10: track 0.00 -> 162.2 mm, vias 0 -> 2
- net /CLOCK_INV: track 0.00 -> 159.9 mm, vias 0 -> 2
- net /a9: track 0.00 -> 152.1 mm, vias 0 -> 2
- net /a8: track 0.00 -> 141.9 mm, vias 0 -> 2
- net CLOCK_IN_PIN: track 0.00 -> 140.8 mm, vias 0 -> 4
- net /a7: track 0.00 -> 131.7 mm, vias 0 -> 2
- net /a6: track 0.00 -> 121.6 mm, vias 0 -> 2
- net A14: track 0.00 -> 119.8 mm, vias 0 -> 2
- net /a5: track 0.00 -> 112.3 mm, vias 0 -> 2
- net /a4: track 0.00 -> 103.5 mm, vias 0 -> 2
- net RESET_PIN: track 0.00 -> 90.9 mm, vias 0 -> 2
- net /a2: track 0.00 -> 83.9 mm, vias 0 -> 2
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Other:
- board size 76 x 119.7 mm -> 114.1 x 114.6 mm

Commit message: Done
Parts:
- moved SW1 27.7 mm to (20.6, 122.6), turned to 90 degrees
- moved R3 18.0 mm to (43.2, 96.5), turned to -90 degrees
- moved C5 6.54 mm to (25.4, 109.2), turned to 180 degrees
Routing:
- net GND: track 320.4 -> 345.0 mm
- net Net-(C5-Pad1): track 30.5 -> 44.7 mm

Commit message: Fix: cpu
Parts:
- added J9: Conn_01x02_Male, Connector_PinHeader_2.54mm:PinHeader_1x02_P2.54mm_Vertical, F.Cu at (111.8, 25.4)
Connections:
- U1 pad 37: CLOCK_IN_PIN -> Net-(U1-Pad37)
Routing:
- net Net-(U1-Pad37): track 0.00 -> 54.0 mm, vias 0 -> 2
- net CLOCK_IN_PIN: track 140.8 -> 129.1 mm, vias 4 -> 2
- net RESET_PIN: track 90.9 -> 89.5 mm
Changed lines of the file:
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@@
   (net 51 "unconnected-(U4-Pad12)")
   (net 52 "/CLOCK_INV")
+  (net 53 "Net-(U1-Pad37)")
   (footprint "Resistor_THT:R_Axial_DIN0411_L9.9mm_D3.6mm_P12.70mm_Horizontal" (layer "F.Cu")
     (at 43.18 96.52 -90)
@@
     )
   )
+  (footprint "Connector_PinHeader_2.54mm:PinHeader_1x02_P2.54mm_Vertical" (layer "F.Cu")
+    (at 111.76 25.4)
+    (descr "Through hole straight pin header, 1x02, 2.54mm pitch, single row")
+    (tags "Through hole pin header THT 1x02 2.54mm single row")
+    (property "Sheetfile" "cpu.kicad_sch")
+    (property "Sheetname" "")
+    (attr through_hole)
+    (fp_text reference "J9" (at 0 -2.33) (layer "F.SilkS")
+      (effects (font (size 1 1) (thickness 0.15)))
+    )
+    (fp_text value "Conn_01x02_Male" (at 0 4.87) (layer "F.Fab")
+      (effects (font (size 1 1) (thickness 0.15)))
+    )
+    (fp_text user "${REFERENCE}" (at 0 1.27 90) (layer "F.Fab")
+      (effects (font (size 1 1) (thickness 0.15)))
+    )
+    (fp_line (start -1.33 1.27) (end 1.33 1.27) (layer "F.SilkS") (width 0.12))
+    (fp_line (start -1.33 -1.33) (end 0 -1.33) (layer "F.SilkS") (width 0.12))
+    (fp_line (start -1.33 3.87) (end 1.33 3.87) (layer "F.SilkS") (width 0.12))
+    (fp_line (start -1.33 0) (end -1.33 -1.33) (layer "F.SilkS") (width 0.12))
+    (fp_line (start -1.33 1.27) (end -1.33 3.87) (layer "F.SilkS") (width 0.12))
+    (fp_line (start 1.33 1.27) (end 1.33 3.87) (layer "F.SilkS") (width 0.12))
+    (fp_line (start 1.8 -1.8) (end -1.8 -1.8) (layer "F.CrtYd") (width 0.05))
+    (fp_line (start -1.8 -1.8) (end -1.8 4.35) (layer "F.CrtYd") (width 0.05))
+    (fp_line (start -1.8 4.35) (end 1.8 4.35) (layer "F.CrtYd") (width 0.05))
+    (fp_line (start 1.8 4.35) (end 1.8 -1.8) (layer "F.CrtYd") (width 0.05))
+    (fp_line (start 1.27 3.81) (end -1.27 3.81) (layer "F.Fab") (width 0.1))
+    (fp_line (start -1.27 3.81) (end -1.27 -0.635) (layer "F.Fab") (width 0.1))
+    (fp_line (start 1.27 -1.27) (end 1.27 3.81) (layer "F.Fab") (width 0.1))
+    (fp_line (start -0.635 -1.27) (end 1.27 -1.27) (layer "F.Fab") (width 0.1))
+    (fp_line (start -1.27 -0.635) (end -0.635 -1.27) (layer "F.Fab") (width 0.1))
+    (pad "1" thru_hole rect locked (at 0 0) (size 1.7 1.7) (drill 1) (layers *.Cu *.Mask)
+      (net 8 "CLOCK_IN_PIN") (pinfunction "Pin_1") (pintype "passive"))
+    (pad "2" thru_hole oval locked (at 0 2.54) (size 1.7 1.7) (drill 1) (layers *.Cu *.Mask)
+      (net 53 "Net-(U1-Pad37)") (pinfunction "Pin_2") (pintype "passive"))
+    (model "${KICAD6_3DMODEL_DIR}/Connector_PinHeader_2.54mm.3dshapes/PinHeader_1x02_P2.54mm_Vertical.wrl"
+      (offset (xyz 0 0 0))
+      (scale (xyz 1 1 1))
+      (rotate (xyz 0 0 0))
+    )
+  )
   (footprint "Resistor_THT:R_Axial_DIN0207_L6.3mm_D2.5mm_P10.16mm_Horizontal" (layer "F.Cu")
     (at 89.028723 109.29478 -90)
@@
       (net 2 "+5V") (pinfunction "BE") (pintype "input"))
     (pad "37" thru_hole oval locked (at 15.24 7.62) (size 2.4 1.6) (drill 0.8) (layers *.Cu *.Mask)
-      (net 8 "CLOCK_IN_PIN") (pinfunction "ϕ0") (pintype "input"))
+      (net 53 "Net-(U1-Pad37)") (pinfunction "ϕ0") (pintype "input"))
     (pad "38" thru_hole oval locked (at 15.24 5.08) (size 2.4 1.6) (drill 0.8) (layers *.Cu *.Mask)
       (net 25 "unconnected-(U1-Pad38)") (pinfunction "~{SO}") (pintype "input+no_connect"))
@@
   (segment (start 83.948723 109.32978) (end 86.598503 106.68) (width 1.5) (layer "B.Cu") (net 7))
   (segment (start 91.498943 106.68) (end 94.108723 109.28978) (width 1.5) (layer "B.Cu") (net 7))
-  (segment (start 119.38 45.72) (end 87.937804 45.72) (width 1.5) (layer "F.Cu") (net 8))
   (segment (start 101.6 106.68) (end 101.6 116.84) (width 1.5) (layer "F.Cu") (net 8))
   (via (at 101.6 106.68) (size 1.5) (drill 0.4) (layers "F.Cu" "B.Cu") (net 8))
-  (via (at 119.38 45.72) (size 1.5) (drill 0.4) (layers "F.Cu" "B.Cu") (net 8))
-  (via (at 87.937804 45.72) (size 1.5) (drill 0.4) (layers "F.Cu" "B.Cu") (net 8))
   (via (at 101.6 116.84) (size 1.5) (drill 0.4) (layers "F.Cu" "B.Cu") (net 8))
-  (segment (start 87.937804 47.942196) (end 87.62 48.26) (width 1.5) (layer "B.Cu") (net 8))
-  (segment (start 124.46 101.6) (end 119.38 106.68) (width 1.5) (layer "B.Cu") (net 8))
+  (segment (start 124.46 35.56) (end 114.3 25.4) (width 1.5) (layer "B.Cu") (net 8))
   (segment (start 101.6 116.84) (end 99.188723 119.251277) (width 1.5) (layer "B.Cu") (net 8))
-  (segment (start 87.937804 45.72) (end 87.937804 47.942196) (width 1.5) (layer "B.Cu") (net 8))
   (segment (start 99.188723 119.251277) (end 99.188723 119.44978) (width 1.5) (layer "B.Cu") (net 8))
-  (segment (start 119.38 45.72) (end 124.46 50.8) (width 1.5) (layer "B.Cu") (net 8))
   (segment (start 101.733723 116.90478) (end 105.548723 116.90478) (width 1.5) (layer "B.Cu") (net 8))
+  (segment (start 124.46 101.6) (end 124.46 35.56) (width 1.5) (layer "B.Cu") (net 8))
+  (segment (start 119.38 106.68) (end 124.46 101.6) (width 1.5) (layer "B.Cu") (net 8))
   (segment (start 99.188723 119.44978) (end 101.733723 116.90478) (width 1.5) (layer "B.Cu") (net 8))
-  (segment (start 124.46 50.8) (end 124.46 101.6) (width 1.5) (layer "B.Cu") (net 8))
-  (segment (start 119.38 106.68) (end 101.6 106.68) (width 1.5) (layer "B.Cu") (net 8))
-  (segment (start 87.62 48.26) (end 85.08 48.26) (width 1.5) (layer "B.Cu") (net 8))
+  (segment (start 101.6 106.68) (end 119.38 106.68) (width 1.5) (layer "B.Cu") (net 8))
+  (segment (start 114.3 25.4) (end 111.76 25.4) (width 1.5) (layer "B.Cu") (net 8))
   (segment (start 99.06 99.06) (end 99.06 93.98) (width 1.5) (layer "F.Cu") (net 9))
   (via (at 99.06 99.06) (size 1.5) (drill 0.4) (layers "F.Cu" "B.Cu") (net 9))
@@
   (segment (start 118.042081 93.98) (end 116.84 93.98) (width 1.5) (layer "B.Cu") (net 13))
   (segment (start 101.6 101.6) (end 116.84 101.6) (width 1.5) (layer "B.Cu") (net 13))
-  (segment (start 110.48 43.18) (end 87.62 43.18) (width 1.5) (layer "F.Cu") (net 14))
+  (segment (start 111.76 43.18) (end 87.62 43.18) (width 1.5) (layer "F.Cu") (net 14))
   (via (at 87.62 43.18) (size 1.5) (drill 0.4) (layers "F.Cu" "B.Cu") (net 14))
-  (via (at 110.48 43.18) (size 1.5) (drill 0.4) (layers "F.Cu" "B.Cu") (net 14))
-  (segment (start 111.76 50.8) (end 111.76 43.18) (width 1.5) (layer "B.Cu") (net 14))
+  (via (at 111.76 43.18) (size 1.5) (drill 0.4) (layers "F.Cu" "B.Cu") (net 14))
   (segment (start 85.08 43.18) (end 87.62 43.18) (width 1.5) (layer "B.Cu") (net 14))
   (segment (start 109.22 88.9) (end 109.22 81.28) (width 1.5) (layer "B.Cu") (net 14))
@@
   (segment (start 113.03 50.8) (end 111.76 50.8) (width 1.5) (layer "B.Cu") (net 14))
   (segment (start 105.4 88.9) (end 109.22 88.9) (width 1.5) (layer "B.Cu") (net 14))
-  (segment (start 111.76 43.18) (end 110.48 43.18) (width 1.5) (layer "B.Cu") (net 14))
+  (segment (start 111.76 43.18) (end 111.76 50.8) (width 1.5) (layer "B.Cu") (net 14))
   (segment (start 109.22 81.28) (end 115.349069 75.150931) (width 1.5) (layer "B.Cu") (net 14))
-  (segment (start 110.48 40.64) (end 87.62 40.64) (width 1.5) (layer "F.Cu") (net 15))
+  (segment (start 111.76 40.64) (end 87.62 40.64) (width 1.5) (layer "F.Cu") (net 15))
   (via (at 87.62 40.64) (size 1.5) (drill 0.4) (layers "F.Cu" "B.Cu") (net 15))
-  (via (at 110.48 40.64) (size 1.5) (drill 0.4) (layers "F.Cu" "B.Cu") (net 15))
-  (segment (start 115.657984 47.077984) (end 119.38 50.8) (width 1.5) (layer "B.Cu") (net 15))
-  (segment (start 110.48 40.64) (end 115.657984 40.64) (width 1.5) (layer "B.Cu") (net 15))
-  (segment (start 115.657984 40.64) (end 115.657984 47.077984) (width 1.5) (layer "B.Cu") (net 15))
-  (segment (start 119.38 50.8) (end 119.38 86.36) (width 1.5) (layer "B.Cu") (net 15))
-  (segment (start 110.48 40.64) (end 110.48 36.84) (width 1.5) (layer "B.Cu") (net 15))
+  (via (at 111.76 40.64) (size 1.5) (drill 0.4) (layers "F.Cu" "B.Cu") (net 15))
+  (segment (start 111.76 40.64) (end 114.3 40.64) (width 1.5) (layer "B.Cu") (net 15))
+  (segment (start 111.76 40.64) (end 111.76 35.56) (width 1.5) (layer "B.Cu") (net 15))
+  (segment (start 119.38 53.34) (end 119.38 86.36) (width 1.5) (layer "B.Cu") (net 15))
+  (segment (start 114.3 48.26) (end 119.38 53.34) (width 1.5) (layer "B.Cu") (net 15))
+  (segment (start 116.84 88.9) (end 113.02 88.9) (width 1.5) (layer "B.Cu") (net 15))
+  (segment (start 114.3 40.64) (end 114.3 48.26) (width 1.5) (layer "B.Cu") (net 15))
   (segment (start 85.08 40.64) (end 87.62 40.64) (width 1.5) (layer "B.Cu") (net 15))
-  (segment (start 116.84 88.9) (end 113.02 88.9) (width 1.5) (layer "B.Cu") (net 15))
-  (segment (start 110.48 36.84) (end 111.76 35.56) (width 1.5) (layer "B.Cu") (net 15))
   (segment (start 119.38 86.36) (end 116.84 88.9) (width 1.5) (layer "B.Cu") (net 15))
   (segment (start 87.62 55.88) (end 111.76 55.88) (width 1.5) (layer "F.Cu") (net 16))
@@
   (segment (start 43.16 102.88) (end 48.27 102.88) (width 1.5) (layer "B.Cu") (net 52))
   (segment (start 116.034606 86.36) (end 116.036459 86.358147) (width 1.5) (layer "B.Cu") (net 52))
+  (segment (start 116.84 45.72) (end 87.937804 45.72) (width 1.5) (layer "F.Cu") (net 53))
+  (via (at 116.84 45.72) (size 1.5) (drill 0.4) (layers "F.Cu" "B.Cu") (net 53))
+  (via (at 87.937804 45.72) (size 1.5) (drill 0.4) (layers "F.Cu" "B.Cu") (net 53))
+  (segment (start 87.937804 47.942196) (end 87.62 48.26) (width 1.5) (layer "B.Cu") (net 53))
+  (segment (start 116.84 33.02) (end 111.76 27.94) (width 1.5) (layer "B.Cu") (net 53))
+  (segment (start 87.937804 45.72) (end 87.937804 47.942196) (width 1.5) (layer "B.Cu") (net 53))
+  (segment (start 116.84 45.72) (end 116.84 33.02) (width 1.5) (layer "B.Cu") (net 53))
+  (segment (start 87.62 48.26) (end 85.08 48.26) (width 1.5) (layer "B.Cu") (net 53))
 )

Commit message: Fit cpu
Parts:
- moved J9 38.1 mm to (111.8, 63.5), turned to 180 degrees
- moved C6 33.2 mm to (88.9, 132.1)
- moved Y1 30.9 mm to (70.9, 122.0)
- moved C7 30.9 mm to (55.8, 132.1)
- moved C8 30.9 mm to (55.8, 124.5)
- moved R4 30.9 mm to (60.9, 122.0)
- moved U4 30.9 mm to (77.4, 122.0)
- moved C9 30.9 mm to (71.0, 132.1)
- moved R5 30.9 mm to (65.9, 132.1)
- moved SW1 29.6 mm to (46.4, 137.2), turned to 180 degrees
- moved C2 25.9 mm to (99.1, 121.9), turned to 0 degrees
- moved J8 25.5 mm to (109.2, 83.8)
- moved C5 21.3 mm to (40.6, 124.2), turned to 0 degrees
- moved U2 19.9 mm to (96.5, 99.1)
- moved J5 19.3 mm to (109.2, 109.2)
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Routing:
- net +5V: track 300.4 -> 454.8 mm, vias 10 -> 7
- net /a11: track 171.6 -> 77.5 mm, vias 2 -> 0
- net /a10: track 162.2 -> 72.4 mm, vias 2 -> 0
- net /a9: track 152.1 -> 78.6 mm
- net /a7: track 131.7 -> 75.5 mm
- net /a6: track 121.6 -> 75.5 mm
- net /a8: track 141.9 -> 97.9 mm, vias 2 -> 4
- net /a5: track 112.3 -> 75.5 mm
- net RESET_PIN: track 89.5 -> 124.9 mm
- net /CLOCK_INV: track 159.9 -> 124.8 mm, vias 2 -> 4
- net A14: track 119.8 -> 149.0 mm, vias 2 -> 0
- net /a4: track 103.5 -> 75.5 mm
- net CLOCK_OUT_PIN: track 81.0 -> 107.5 mm, vias 2 -> 4
- net CLOCK_IN_PIN: track 129.1 -> 109.4 mm, vias 2 -> 4
- net Net-(U1-Pad37): track 54.0 -> 37.7 mm
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Other:
- board size 114.1 x 114.6 mm -> 90.1 x 130.6 mm
